Commit message: tested jamal with RL

File: resources/robots/jamal/urdf/jamal2_v5.urdf (robot description, URDF)
Before this commit: robot jamal2_v5, 19 links, 18 joints
Joints:
- joint FL_foot_joint: origin xyz=-0.00157691666386468 5.00000000003276E-05 -0.24800624908566 rpy=0 0 0 -> xyz=-0.00157691666386468 5.00000000003276E-05 -0.23 rpy=0 0 0
- joint FR_foot_joint: origin xyz=-0.0016311444601869 -5.00000000001333E-05 -0.248006659789989 rpy=0 0 0 -> xyz=-0.0016311444601869 -5.00000000001333E-05 -0.23 rpy=0 0 0
- joint RL_foot_joint: origin xyz=0.000550115239932258 5.00000000001888E-05 -0.248000939223794 rpy=0 0 0 -> xyz=0.000550115239932258 5.00000000001888E-05 -0.23 rpy=0 0 0
- joint RR_foot_joint: origin xyz=0.00181474156111877 -5.000000000005E-05 -0.248008147336944 rpy=0 0 0 -> xyz=0.00181474156111877 -5.000000000005E-05 -0.23 rpy=0 0 0
