Commit message: testing RL with jamal

File: resources/robots/jamal/urdf/jamal_inverted.urdf (robot description, URDF)
Before this commit: robot robot, 17 links, 16 joints
Links:
- removed link LF_FOOT
- removed link LH_FOOT
- removed link RF_FOOT
- removed link RH_FOOT
- added link LF_foot, mass 0.06; collision sphere radius=0.02; visual mesh filename=../dae/foot.dae
- added link LH_foot, mass 0.06; collision sphere radius=0.02; visual mesh filename=../dae/foot.dae
- added link RF_foot, mass 0.06; collision sphere radius=0.02; visual mesh filename=../dae/foot.dae
- added link RH_foot, mass 0.06; collision sphere radius=0.02; visual mesh filename=../dae/foot.dae
- added link imu, mass 0
- link LF_calf: geometry collision box size=0.23 0.016 0.016; visual mesh filename=../dae/calf.dae scale=1 1 1
- link LH_calf: geometry collision box size=0.23 0.016 0.016; visual mesh filename=../dae/calf.dae scale=1 1 1
- link RF_calf: geometry collision box size=0.23 0.016 0.016; visual mesh filename=../dae/calf.dae scale=1 1 1
- link RH_calf: geometry collision box size=0.23 0.016 0.016; visual mesh filename=../dae/calf.dae scale=1 1 1
- link base: geometry collision box size=0.3762 0.2 0.114; visual mesh filename=../dae/base.dae scale=1 1 1
Joints:
- added joint imu_joint: type fixed, parent base, child imu, origin xyz=-0.02557 0 0.04232 rpy=0 0 0, axis 0 0 0
- joint FL_calf_joint: limit lower=-2.818 upper=2.818 effort=100 velocity=8 -> lower=-2.62 upper=-0.78 effort=100 velocity=30
- joint FL_hip_joint: limit lower=-0.863 upper=0.863 effort=100 velocity=8 -> lower=-0.863 upper=0.863 effort=100 velocity=30
- joint FL_thigh_joint: limit lower=-1.57 upper=1.57 effort=100 velocity=8 -> lower=0.0 upper=1.57 effort=100 velocity=30
- joint FR_calf_joint: limit lower=-2.818 upper=2.818 effort=100 velocity=8 -> lower=-2.62 upper=-0.78 effort=100 velocity=30
- joint FR_hip_joint: limit lower=-0.863 upper=0.863 effort=100 velocity=8 -> lower=-0.863 upper=0.863 effort=100 velocity=30
- joint FR_thigh_joint: limit lower=-1.57 upper=1.57 effort=100 velocity=8 -> lower=0.0 upper=1.57 effort=100 velocity=30
- joint LF_foot_fixed: child LF_FOOT -> LF_foot
- joint LH_foot_fixed: child LH_FOOT -> LH_foot
- joint RF_foot_fixed: child RF_FOOT -> RF_foot
- joint RH_foot_fixed: child RH_FOOT -> RH_foot
- joint RL_calf_joint: limit lower=-2.818 upper=2.818 effort=100 velocity=8 -> lower=0.78 upper=2.62 effort=100 velocity=30
- joint RL_hip_joint: limit lower=-0.863 upper=0.863 effort=100 velocity=8 -> lower=-0.863 upper=0.863 effort=100 velocity=30
- joint RL_thigh_joint: limit lower=-1.57 upper=0.0 effort=100 velocity=8 -> lower=-1.57 upper=0.0 effort=100 velocity=30
- joint RR_calf_joint: limit lower=-2.818 upper=2.818 effort=100 velocity=8 -> lower=0.78 upper=2.62 effort=100 velocity=30
- joint RR_hip_joint: limit lower=-0.863 upper=0.863 effort=100 velocity=8 -> lower=-0.863 upper=0.863 effort=100 velocity=30
- joint RR_thigh_joint: limit lower=-1.57 upper=0.0 effort=100 velocity=8 -> lower=-1.57 upper=0.0 effort=100 velocity=30

Commit message: best walking policy trained

File: resources/robots/jamal/urdf/jamal_inverted.urdf (robot description, URDF)
Before this commit: robot jamal_description, 18 links, 17 joints
Joints:
- joint FL_hip_joint: limit lower=-0.863 upper=0.863 effort=100 velocity=8 -> lower=-0.4 upper=0.4 effort=100 velocity=8
- joint FR_hip_joint: limit lower=-0.863 upper=0.863 effort=100 velocity=8 -> lower=-0.4 upper=0.4 effort=100 velocity=8
- joint RL_hip_joint: limit lower=-0.863 upper=0.863 effort=100 velocity=8 -> lower=-0.4 upper=0.4 effort=100 velocity=8
- joint RR_hip_joint: limit lower=-0.863 upper=0.863 effort=100 velocity=8 -> lower=-0.4 upper=0.4 effort=100 velocity=8
