Commit message: walking tested on jamal backward bend

File: resources/robots/go2/urdf/go2_tested.urdf (robot description, URDF)
Before this commit: robot go2_description, 18 links, 17 joints
Links:
- added link FL_calflower; collision cylinder length=0.065 radius=0.011
- added link FL_calflower1; collision cylinder length=0.03 radius=0.0155
- added link FR_calflower; collision cylinder length=0.065 radius=0.011
- added link FR_calflower1; collision cylinder length=0.03 radius=0.0155
- added link Head_lower, mass 0.001; collision sphere radius=0.047
- added link Head_upper, mass 0.001; collision cylinder length=0.09 radius=0.05
- added link RL_calflower; collision cylinder length=0.065 radius=0.011
- added link RL_calflower1; collision cylinder length=0.03 radius=0.0155
- added link RR_calflower; collision cylinder length=0.065 radius=0.011
- added link RR_calflower1; collision cylinder length=0.03 radius=0.0155
- added link radar, mass 0
- link FL_calf: mass 0.12879265462489 -> 0.154; geometry collision cylinder length=0.12 radius=0.012; visual mesh filename=../dae/calf.dae
- link FL_foot: mass 0.06 -> 0.04
- link FL_hip: mass 0.933762854916433 -> 0.678
- link FL_thigh: mass 1.32134262348697 -> 1.152; geometry collision box size=0.11 0.0245 0.034; visual mesh filename=../dae/thigh.dae
- link FR_calf: mass 0.12879265462489 -> 0.154; geometry collision cylinder length=0.12 radius=0.013; visual mesh filename=../dae/calf_mirror.dae
- link FR_foot: mass 0.06 -> 0.04; geometry collision sphere radius=0.022; visual mesh filename=../dae/foot.dae
- link FR_hip: mass 0.933762854916433 -> 0.678
- link FR_thigh: mass 1.32134262348697 -> 1.152; geometry collision box size=0.11 0.0245 0.034; visual mesh filename=../dae/thigh_mirror.dae
- link RL_calf: mass 0.12879265462489 -> 0.154; geometry collision cylinder length=0.12 radius=0.013; visual mesh filename=../dae/calf.dae
- link RL_foot: mass 0.06 -> 0.04; geometry collision sphere radius=0.022; visual mesh filename=../dae/foot.dae
- link RL_hip: mass 0.933762854916433 -> 0.678
- link RL_thigh: mass 1.32134262348697 -> 1.152; geometry collision box size=0.11 0.0245 0.034; visual mesh filename=../dae/thigh.dae
- link RR_calf: mass 0.12879265462489 -> 0.154; geometry collision cylinder length=0.12 radius=0.013; visual mesh filename=../dae/calf_mirror.dae
- link RR_foot: mass 0.06 -> 0.04; geometry collision sphere radius=0.022; visual mesh filename=../dae/foot.dae
- link RR_hip: mass 0.933762854916433 -> 0.678
- link RR_thigh: mass 1.32134262348697 -> 1.152; geometry collision box size=0.11 0.0245 0.034; visual mesh filename=../dae/thigh_mirror.dae
- link base: mass 12.8185384756311 -> 6.921; geometry collision box size=0.3762 0.0935 0.114; visual mesh filename=../dae/base.dae
Joints:
- added joint FL_calflower1_joint: type fixed, parent FL_calflower, child FL_calflower1, origin xyz=-0.01 0 -0.04 rpy=0 0.48 0, axis 0 0 0
- added joint FL_calflower_joint: type fixed, parent FL_calf, child FL_calflower, origin xyz=0.020 0 -0.148 rpy=0 0.05 0, axis 0 0 0
- added joint FR_calflower1_joint: type fixed, parent FR_calflower, child FR_calflower1, origin xyz=-0.01 0 -0.04 rpy=0 0.48 0, axis 0 0 0
- added joint FR_calflower_joint: type fixed, parent FR_calf, child FR_calflower, origin xyz=0.020 0 -0.148 rpy=0 0.05 0, axis 0 0 0
- added joint Head_lower_joint: type fixed, parent Head_upper, child Head_lower, origin xyz=0.008 0 -0.07 rpy=0 0 0, axis 0 0 0
- added joint Head_upper_joint: type fixed, parent base, child Head_upper, origin xyz=0.285 0 0.01 rpy=0 0 0, axis 0 0 0
- added joint RL_calflower1_joint: type fixed, parent RL_calflower, child RL_calflower1, origin xyz=-0.01 0 -0.04 rpy=0 0.48 0, axis 0 0 0
- added joint RL_calflower_joint: type fixed, parent RL_calf, child RL_calflower, origin xyz=0.020 0 -0.148 rpy=0 0.05 0, axis 0 0 0
- added joint RR_calflower1_joint: type fixed, parent RR_calflower, child RR_calflower1, origin xyz=-0.01 0 -0.04 rpy=0 0.48 0, axis 0 0 0
- added joint RR_calflower_joint: type fixed, parent RR_calf, child RR_calflower, origin xyz=0.020 0 -0.148 rpy=0 0.05 0, axis 0 0 0
- added joint radar_joint: type fixed, parent base, child radar, origin xyz=0.28945 0 -0.046825 rpy=0 2.8782 0, axis 0 0 0
- joint FL_calf_joint: limit lower=-2.7227 upper=-0.83776 effort=100 velocity=20.07 -> lower=-2.7227 upper=-0.83776 effort=35.55 velocity=20.07; origin xyz=0 0 -0.225 rpy=0 0 0 -> xyz=0 0 -0.213 rpy=0 0 0
- joint FL_foot_joint: origin xyz=0 0 -0.23 rpy=0 0 0 -> xyz=0 0 -0.213 rpy=0 0 0
- joint FL_hip_joint: limit lower=-1.0472 upper=1.0472 effort=100 velocity=30.1 -> lower=-1.0472 upper=1.0472 effort=23.7 velocity=30.1; origin xyz=0.2699 0.08028 0 rpy=0 0 0 -> xyz=0.1934 0.0465 0 rpy=0 0 0
- joint FL_thigh_joint: limit lower=-1.5708 upper=3.4907 effort=100 velocity=30.1 -> lower=-1.5708 upper=3.4907 effort=23.7 velocity=30.1; origin xyz=0 0.10755 0 rpy=0 0 0 -> xyz=0 0.0955 0 rpy=0 0 0
- joint FR_calf_joint: limit lower=-2.7227 upper=-0.83776 effort=100 velocity=20.07 -> lower=-2.7227 upper=-0.83776 effort=35.55 velocity=20.07; origin xyz=0 0 -0.225 rpy=0 0 0 -> xyz=0 0 -0.213 rpy=0 0 0
- joint FR_foot_joint: origin xyz=0 0 -0.23 rpy=0 0 0 -> xyz=0 0 -0.213 rpy=0 0 0
- joint FR_hip_joint: limit lower=-1.0472 upper=1.0472 effort=100 velocity=30.1 -> lower=-1.0472 upper=1.0472 effort=23.7 velocity=30.1; origin xyz=0.2699 -0.08028 0 rpy=0 0 0 -> xyz=0.1934 -0.0465 0 rpy=0 0 0
- joint FR_thigh_joint: limit lower=-1.5708 upper=3.4907 effort=100 velocity=30.1 -> lower=-1.5708 upper=3.4907 effort=23.7 velocity=30.1; origin xyz=0 -0.10755 0 rpy=0 0 0 -> xyz=0 -0.0955 0 rpy=0 0 0
- joint RL_calf_joint: limit lower=-2.7227 upper=-0.83776 effort=100 velocity=20.07 -> lower=-2.7227 upper=-0.83776 effort=35.55 velocity=20.07; origin xyz=0 0 -0.225 rpy=0 0 0 -> xyz=0 0 -0.213 rpy=0 0 0
- joint RL_foot_joint: origin xyz=0 0 -0.23 rpy=0 0 0 -> xyz=0 0 -0.213 rpy=0 0 0
- joint RL_hip_joint: limit lower=-1.0472 upper=1.0472 effort=100 velocity=30.1 -> lower=-1.0472 upper=1.0472 effort=23.7 velocity=30.1; origin xyz=-0.2699 0.08028 0 rpy=0 0 0 -> xyz=-0.1934 0.0465 0 rpy=0 0 0
- joint RL_thigh_joint: limit lower=-0.5236 upper=4.5379 effort=100 velocity=30.1 -> lower=-0.5236 upper=4.5379 effort=23.7 velocity=30.1; origin xyz=0 0.10755 0 rpy=0 0 0 -> xyz=0 0.0955 0 rpy=0 0 0
- joint RR_calf_joint: limit lower=-2.7227 upper=-0.83776 effort=100 velocity=20.07 -> lower=-2.7227 upper=-0.83776 effort=35.55 velocity=20.07; origin xyz=0 0 -0.225 rpy=0 0 0 -> xyz=0 0 -0.213 rpy=0 0 0
- joint RR_foot_joint: origin xyz=0 0 -0.23 rpy=0 0 0 -> xyz=0 0 -0.213 rpy=0 0 0
- joint RR_hip_joint: limit lower=-1.0472 upper=1.0472 effort=100 velocity=30.1 -> lower=-1.0472 upper=1.0472 effort=23.7 velocity=30.1; origin xyz=-0.2699 -0.08028 0 rpy=0 0 0 -> xyz=-0.1934 -0.0465 0 rpy=0 0 0
- joint RR_thigh_joint: limit lower=-0.5236 upper=4.5379 effort=100 velocity=30.1 -> lower=-0.5236 upper=4.5379 effort=23.7 velocity=30.1; origin xyz=0 -0.10755 0 rpy=0 0 0 -> xyz=0 -0.0955 0 rpy=0 0 0

File: resources/robots/jamal/urdf/jamal.urdf (robot description, URDF)
Before this commit: robot go2_description, 18 links, 17 joints
Links:
- link FR_calf: geometry collision box size=0.23 0.016 0.016; visual mesh filename=../dae/calf.dae
- link RR_calf: geometry collision box size=0.23 0.016 0.016; visual mesh filename=../dae/calf.dae
Joints:
- joint FL_hip_joint: limit lower=-1.0472 upper=1.0472 effort=100 velocity=30.1 -> lower=-0.53 upper=0.53 effort=100 velocity=8
- joint FL_thigh_joint: limit lower=-1.5708 upper=3.4907 effort=100 velocity=30.1 -> lower=-1.5708 upper=3.4907 effort=100 velocity=8
- joint FR_hip_joint: limit lower=-1.0472 upper=1.0472 effort=100 velocity=30.1 -> lower=-0.53 upper=0.53 effort=100 velocity=8
- joint FR_thigh_joint: limit lower=-1.5708 upper=3.4907 effort=100 velocity=30.1 -> lower=-1.5708 upper=3.4907 effort=100 velocity=8
- joint RL_hip_joint: limit lower=-1.0472 upper=1.0472 effort=100 velocity=30.1 -> lower=-0.53 upper=0.53 effort=100 velocity=8
- joint RL_thigh_joint: limit lower=-0.5236 upper=4.5379 effort=100 velocity=30.1 -> lower=-0.5236 upper=4.5379 effort=100 velocity=8
- joint RR_hip_joint: limit lower=-1.0472 upper=1.0472 effort=100 velocity=30.1 -> lower=-0.53 upper=0.53 effort=100 velocity=8
- joint RR_thigh_joint: limit lower=-0.5236 upper=4.5379 effort=100 velocity=30.1 -> lower=-0.5236 upper=4.5379 effort=100 velocity=8

File: resources/robots/jamal/urdf/jamal2_v5.urdf (robot description, URDF)
Before this commit: robot jamal2_v5, 19 links, 18 joints
Links:
- link base: mass 13.2256112448737 -> 12.8185384756311

File: resources/robots/jamal/urdf/jamal_inverted.urdf (robot description, URDF)
Before this commit: robot jamal_description, 18 links, 17 joints
Joints:
- joint FL_calf_joint: limit lower=-2.62 upper=-0.78 effort=100 velocity=30 -> lower=-2.62 upper=-0.78 effort=100 velocity=8
- joint FL_hip_joint: limit lower=-0.863 upper=0.863 effort=100 velocity=30 -> lower=-0.863 upper=0.863 effort=100 velocity=8
- joint FL_thigh_joint: limit lower=0.0 upper=1.57 effort=100 velocity=30 -> lower=0.0 upper=1.57 effort=100 velocity=8
- joint FR_calf_joint: limit lower=-2.62 upper=-0.78 effort=100 velocity=30 -> lower=-2.62 upper=-0.78 effort=100 velocity=8
- joint FR_hip_joint: limit lower=-0.863 upper=0.863 effort=100 velocity=30 -> lower=-0.863 upper=0.863 effort=100 velocity=8
- joint FR_thigh_joint: limit lower=0.0 upper=1.57 effort=100 velocity=30 -> lower=0.0 upper=1.57 effort=100 velocity=8
- joint RL_calf_joint: limit lower=0.78 upper=2.62 effort=100 velocity=30 -> lower=0.78 upper=2.62 effort=100 velocity=8
- joint RL_hip_joint: limit lower=-0.863 upper=0.863 effort=100 velocity=30 -> lower=-0.863 upper=0.863 effort=100 velocity=8
- joint RL_thigh_joint: limit lower=-1.57 upper=0.0 effort=100 velocity=30 -> lower=-1.57 upper=0.0 effort=100 velocity=8
- joint RR_calf_joint: limit lower=0.78 upper=2.62 effort=100 velocity=30 -> lower=0.78 upper=2.62 effort=100 velocity=8
- joint RR_hip_joint: limit lower=-0.863 upper=0.863 effort=100 velocity=30 -> lower=-0.863 upper=0.863 effort=100 velocity=8
- joint RR_thigh_joint: limit lower=-1.57 upper=0.0 effort=100 velocity=30 -> lower=-1.57 upper=0.0 effort=100 velocity=8
